Commit message: [fix]: working version of mobile base

File: urdf/stretch_base.xacro (robot description, xacro)
@@ -34,5 +34,5 @@
         rpy="0 0 0" />
       <mass
-        value="4.3" />
+        value="1.1912" />
       <inertia
         ixx="0.0034667"
@@ -84,5 +84,5 @@
       </geometry>
     </collision>
-    <xacro:default_inertial mass="0.0042721" pos="1.1719E-11 2.0783E-11 0.037544"/>
+    <xacro:default_inertial mass="0.5" pos="1.1719E-11 2.0783E-11 0.037544"/>
   </link>
   <joint
@@ -98,5 +98,5 @@
     <axis
       xyz="0 0 1" />
-    <dynamics damping="${joint_damping}" friction="${joint_friction}" spring_reference="${joint_spring_reference}" spring_stiffness="${joint_spring_stiffness}"/>
+    <!-- <dynamics damping="${joint_damping}" friction="${joint_friction}" spring_reference="${joint_spring_reference}" spring_stiffness="${joint_spring_stiffness}"/> -->
   </joint>
   <link
@@ -121,5 +121,5 @@
       </geometry>
     </collision>
-    <xacro:default_inertial mass="0.0042721" pos="-2.0783E-11 -1.1719E-11 -0.037544"/>
+    <xacro:default_inertial mass="0.5" pos="-2.0783E-11 -1.1719E-11 -0.037544"/>
   </link>
   <joint
@@ -135,5 +135,5 @@
     <axis
       xyz="0 0 1" />
-    <dynamics damping="${joint_damping}" friction="${joint_friction}" spring_reference="${joint_spring_reference}" spring_stiffness="${joint_spring_stiffness}"/>
+    <!-- <dynamics damping="${joint_damping}" friction="${joint_friction}" spring_reference="${joint_spring_reference}" spring_stiffness="${joint_spring_stiffness}"/> -->
   </joint>
   <link name="caster_link">

Commit message: [fix]: Changed to default values for mobile base

File: urdf/stretch_base.xacro (robot description, xacro)
@@ -2,6 +2,6 @@
 <robot xmlns:xacro="http://www.ros.org/wiki/xacro" name="stretch_base">
   <xacro:property name="M_PI" value="3.1415926535897931" />
-  <xacro:property name="joint_damping" value="21.75"/>
-  <xacro:property name="joint_friction" value="10.48"/>
+  <xacro:property name="joint_damping" value="0"/>
+  <xacro:property name="joint_friction" value="0"/>
   <xacro:property name="joint_spring_stiffness" value="0"/>
   <xacro:property name="joint_spring_reference" value="0"/>
@@ -19,10 +19,10 @@
       <mass value="${mass}" />
       <inertia
-        ixx="5.4E-05"
+        ixx="0.01"
         ixy="0"
         ixz="0"
-        iyy="5.4E-05"
+        iyy="0.01"
         iyz="0"
-        izz="5.4E-05" />
+        izz="0.01" />
     </inertial>
   </xacro:macro>
@@ -84,5 +84,5 @@
       </geometry>
     </collision>
-    <xacro:default_inertial mass="0.5" pos="1.1719E-11 2.0783E-11 0.037544"/>
+    <xacro:default_inertial mass="0.0042721" pos="1.1719E-11 2.0783E-11 0.037544"/>
   </link>
   <joint
@@ -98,5 +98,5 @@
     <axis
       xyz="0 0 1" />
-    <!-- <dynamics damping="${joint_damping}" friction="${joint_friction}" spring_reference="${joint_spring_reference}" spring_stiffness="${joint_spring_stiffness}"/> -->
+    <dynamics damping="${joint_damping}" friction="${joint_friction}" spring_reference="${joint_spring_reference}" spring_stiffness="${joint_spring_stiffness}"/>
   </joint>
   <link
@@ -121,5 +121,5 @@
       </geometry>
     </collision>
-    <xacro:default_inertial mass="0.5" pos="-2.0783E-11 -1.1719E-11 -0.037544"/>
+    <xacro:default_inertial mass="0.0042721" pos="-2.0783E-11 -1.1719E-11 -0.037544"/>
   </link>
   <joint
@@ -135,5 +135,5 @@
     <axis
       xyz="0 0 1" />
-    <!-- <dynamics damping="${joint_damping}" friction="${joint_friction}" spring_reference="${joint_spring_reference}" spring_stiffness="${joint_spring_stiffness}"/> -->
+    <dynamics damping="${joint_damping}" friction="${joint_friction}" spring_reference="${joint_spring_reference}" spring_stiffness="${joint_spring_stiffness}"/>
   </joint>
   <link name="caster_link">
