Commit message: [fix]: Changed config file for ros2 controller mobile base

File: urdf/stretch_main.xacro (robot description, xacro)
@@ -2,6 +2,6 @@
 <robot xmlns:xacro="http://www.ros.org/wiki/xacro" name="stretch_main">
   <xacro:property name="M_PI" value="3.1415926535897931" />
-  <xacro:property name="joint_damping" value="21.75"/>
-  <xacro:property name="joint_friction" value="10.48"/>
+  <xacro:property name="joint_damping" value="0"/>
+  <xacro:property name="joint_friction" value="0"/>
   <xacro:property name="joint_spring_stiffness" value="0"/>
   <xacro:property name="joint_spring_reference" value="0"/>
