Commit message: Creation of dev branch

File: urdf/gazebo.urdf.xacro (robot description, xacro)
@@ -29,22 +29,4 @@
     <mu1>0.0</mu1>
     <mu2>0.0</mu2>
-  </gazebo>
-  <gazebo reference="link_aruco_right_base">
-      <material>Gazebo/Black</material>
-  </gazebo>
-  <gazebo reference="link_aruco_left_base">
-      <material>Gazebo/Black</material>
-  </gazebo>
-  <gazebo reference="link_aruco_shoulder">
-      <material>Gazebo/Black</material>
-  </gazebo>
-  <gazebo reference="link_aruco_top_wrist">
-      <material>Gazebo/Black</material>
-  </gazebo>
-  <gazebo reference="link_aruco_inner_wrist">
-      <material>Gazebo/Black</material>
-  </gazebo>
-  <gazebo reference="respeaker_base">
-      <material>Gazebo/Green</material>
   </gazebo>
   <gazebo reference="link_lift">
@@ -138,12 +120,6 @@
       </command_interface>
       <state_interface name="position" />
-    </joint>
-    <transmission name="right_wheel_trans" type="SimpleTransmission">
-        <plugin>transmission_interface/SimpleTransmission</plugin>
-        <actuator name="right_wheel_motor" role="actuator1"/>
-        <joint name="joint_right_wheel" role="joint1">
-            <mechanicalReduction>1</mechanicalReduction>
-        </joint>
-    </transmission>
+      <state_interface name="velocity" />
+    </joint>
     <joint name="joint_left_wheel">
         <command_interface name="velocity">
@@ -152,12 +128,6 @@
         </command_interface>
         <state_interface name="position" />
-    </joint>
-    <transmission name="left_wheel_trans" type="SimpleTransmission">
-        <plugin>transmission_interface/SimpleTransmission</plugin>
-        <actuator name="left_wheel_motor" role="actuator1"/>
-        <joint name="joint_left_wheel" role="joint1">
-            <mechanicalReduction>1</mechanicalReduction>
-        </joint>
-    </transmission>
+        <state_interface name="velocity" />
+    </joint>
     <joint name="joint_lift">
       <command_interface name="position" />
@@ -168,12 +138,4 @@
       <state_interface name="effort" />
     </joint>
-    <transmission name="trans_lift">
-        <plugin>transmission_interface/SimpleTransmission</plugin>
-        <actuator name="motor_lift" role="actuator1"/>
-        <joint name="joint_lift" role="joint1">
-            <mechanical_reduction>1.0</mechanical_reduction>
-            <offset>0.0</offset>
-        </joint>
-    </transmission>
     <joint name="joint_arm_l0">
       <command_interface name="position" />
@@ -184,12 +146,4 @@
       <state_interface name="effort" />
     </joint>
-    <transmission name="trans_arm_l0">
-        <plugin>transmission_interface/SimpleTransmission</plugin>
-        <actuator name="motor_arm_l0" role="actuator1"/>
-        <joint name="joint_arm_l0" role="joint1">
-            <mechanical_reduction>1.0</mechanical_reduction>
-            <offset>0.0</offset>
-        </joint>
-    </transmission>
     <joint name="joint_arm_l1">
       <command_interface name="position" />
@@ -200,12 +154,4 @@
       <state_interface name="effort" />
     </joint>
-    <transmission name="trans_arm_l1">
-        <plugin>transmission_interface/SimpleTransmission</plugin>
-        <actuator name="motor_arm_l1" role="actuator1"/>
-        <joint name="joint_arm_l1" role="joint1">
-            <mechanical_reduction>1.0</mechanical_reduction>
-            <offset>0.0</offset>
-        </joint>
-    </transmission>
     <joint name="joint_arm_l2">
       <command_interface name="position" />
@@ -216,12 +162,4 @@
       <state_interface name="effort" />
     </joint>
-    <transmission name="trans_arm_l2">
-      <plugin>transmission_interface/SimpleTransmission</plugin>
-      <actuator name="motor_arm_l2" role="actuator1"/>
-      <joint name="joint_arm_l2" role="joint1">
-          <mechanical_reduction>1.0</mechanical_reduction>
-          <offset>0.0</offset>
-      </joint>
-    </transmission>
     <joint name="joint_arm_l3">
       <command_interface name="position" />
@@ -232,12 +170,4 @@
       <state_interface name="effort" />
     </joint>
-    <transmission name="trans_arm_l3">
-      <plugin>transmission_interface/SimpleTransmission</plugin>
-      <actuator name="motor_arm_l3" role="actuator1"/>
-      <joint name="joint_arm_l3" role="joint1">
-          <mechanical_reduction>1.0</mechanical_reduction>
-          <offset>0.0</offset>
-      </joint>
-    </transmission>
     <joint name="joint_wrist_yaw">
       <command_interface name="position" />
@@ -248,12 +178,4 @@
       <state_interface name="effort" />
     </joint>
-    <transmission name="trans_wrist_yaw">
-      <plugin>transmission_interface/SimpleTransmission</plugin>
-      <actuator name="motor_wrist_yaw" role="actuator1"/>
-      <joint name="joint_wrist_yaw" role="joint1">
-          <mechanical_reduction>1.0</mechanical_reduction>
-          <offset>0.0</offset>
-      </joint>
-    </transmission>
     <joint name="joint_head_pan">
       <command_interface name="position" />
@@ -264,12 +186,4 @@
       <state_interface name="effort" />
     </joint>
-    <transmission name="trans_head_pan">
-      <plugin>transmission_interface/SimpleTransmission</plugin>
-      <actuator name="motor_head_pan" role="actuator1"/>
-      <joint name="joint_head_pan" role="joint1">
-          <mechanical_reduction>1.0</mechanical_reduction>
-          <offset>0.0</offset>
-      </joint>
-    </transmission>
     <joint name="joint_head_tilt">
       <command_interface name="position" />
@@ -280,12 +194,4 @@
       <state_interface name="effort" />
     </joint>
-    <transmission name="trans_head_tilt">
-      <plugin>transmission_interface/SimpleTransmission</plugin>
-      <actuator name="motor_head_tilt" role="actuator1"/>
-      <joint name="joint_head_tilt" role="joint1">
-          <mechanical_reduction>1.0</mechanical_reduction>
-          <offset>0.0</offset>
-      </joint>
-    </transmission>
   </ros2_control>
   <gazebo>

File: urdf/stretch_main.xacro (robot description, xacro)
@@ -210,5 +210,5 @@
         rpy="0 0 0" />
       <mass
-        value="1.8285" />
+        value="0.18285" />
       <inertia
         ixx="0.0709854511954588"

Commit message: [fix]: wrong pull into branch

File: urdf/gazebo.urdf.xacro (robot description, xacro)
@@ -29,4 +29,22 @@
     <mu1>0.0</mu1>
     <mu2>0.0</mu2>
+  </gazebo>
+  <gazebo reference="link_aruco_right_base">
+      <material>Gazebo/Black</material>
+  </gazebo>
+  <gazebo reference="link_aruco_left_base">
+      <material>Gazebo/Black</material>
+  </gazebo>
+  <gazebo reference="link_aruco_shoulder">
+      <material>Gazebo/Black</material>
+  </gazebo>
+  <gazebo reference="link_aruco_top_wrist">
+      <material>Gazebo/Black</material>
+  </gazebo>
+  <gazebo reference="link_aruco_inner_wrist">
+      <material>Gazebo/Black</material>
+  </gazebo>
+  <gazebo reference="respeaker_base">
+      <material>Gazebo/Green</material>
   </gazebo>
   <gazebo reference="link_lift">
@@ -120,6 +138,12 @@
       </command_interface>
       <state_interface name="position" />
-      <state_interface name="velocity" />
-    </joint>
+    </joint>
+    <transmission name="right_wheel_trans" type="SimpleTransmission">
+        <plugin>transmission_interface/SimpleTransmission</plugin>
+        <actuator name="right_wheel_motor" role="actuator1"/>
+        <joint name="joint_right_wheel" role="joint1">
+            <mechanicalReduction>1</mechanicalReduction>
+        </joint>
+    </transmission>
     <joint name="joint_left_wheel">
         <command_interface name="velocity">
@@ -128,6 +152,12 @@
         </command_interface>
         <state_interface name="position" />
-        <state_interface name="velocity" />
-    </joint>
+    </joint>
+    <transmission name="left_wheel_trans" type="SimpleTransmission">
+        <plugin>transmission_interface/SimpleTransmission</plugin>
+        <actuator name="left_wheel_motor" role="actuator1"/>
+        <joint name="joint_left_wheel" role="joint1">
+            <mechanicalReduction>1</mechanicalReduction>
+        </joint>
+    </transmission>
     <joint name="joint_lift">
       <command_interface name="position" />
@@ -138,4 +168,12 @@
       <state_interface name="effort" />
     </joint>
+    <transmission name="trans_lift">
+        <plugin>transmission_interface/SimpleTransmission</plugin>
+        <actuator name="motor_lift" role="actuator1"/>
+        <joint name="joint_lift" role="joint1">
+            <mechanical_reduction>1.0</mechanical_reduction>
+            <offset>0.0</offset>
+        </joint>
+    </transmission>
     <joint name="joint_arm_l0">
       <command_interface name="position" />
@@ -146,4 +184,12 @@
       <state_interface name="effort" />
     </joint>
+    <transmission name="trans_arm_l0">
+        <plugin>transmission_interface/SimpleTransmission</plugin>
+        <actuator name="motor_arm_l0" role="actuator1"/>
+        <joint name="joint_arm_l0" role="joint1">
+            <mechanical_reduction>1.0</mechanical_reduction>
+            <offset>0.0</offset>
+        </joint>
+    </transmission>
     <joint name="joint_arm_l1">
       <command_interface name="position" />
@@ -154,4 +200,12 @@
       <state_interface name="effort" />
     </joint>
+    <transmission name="trans_arm_l1">
+        <plugin>transmission_interface/SimpleTransmission</plugin>
+        <actuator name="motor_arm_l1" role="actuator1"/>
+        <joint name="joint_arm_l1" role="joint1">
+            <mechanical_reduction>1.0</mechanical_reduction>
+            <offset>0.0</offset>
+        </joint>
+    </transmission>
     <joint name="joint_arm_l2">
       <command_interface name="position" />
@@ -162,4 +216,12 @@
       <state_interface name="effort" />
     </joint>
+    <transmission name="trans_arm_l2">
+      <plugin>transmission_interface/SimpleTransmission</plugin>
+      <actuator name="motor_arm_l2" role="actuator1"/>
+      <joint name="joint_arm_l2" role="joint1">
+          <mechanical_reduction>1.0</mechanical_reduction>
+          <offset>0.0</offset>
+      </joint>
+    </transmission>
     <joint name="joint_arm_l3">
       <command_interface name="position" />
@@ -170,4 +232,12 @@
       <state_interface name="effort" />
     </joint>
+    <transmission name="trans_arm_l3">
+      <plugin>transmission_interface/SimpleTransmission</plugin>
+      <actuator name="motor_arm_l3" role="actuator1"/>
+      <joint name="joint_arm_l3" role="joint1">
+          <mechanical_reduction>1.0</mechanical_reduction>
+          <offset>0.0</offset>
+      </joint>
+    </transmission>
     <joint name="joint_wrist_yaw">
       <command_interface name="position" />
@@ -178,4 +248,12 @@
       <state_interface name="effort" />
     </joint>
+    <transmission name="trans_wrist_yaw">
+      <plugin>transmission_interface/SimpleTransmission</plugin>
+      <actuator name="motor_wrist_yaw" role="actuator1"/>
+      <joint name="joint_wrist_yaw" role="joint1">
+          <mechanical_reduction>1.0</mechanical_reduction>
+          <offset>0.0</offset>
+      </joint>
+    </transmission>
     <joint name="joint_head_pan">
       <command_interface name="position" />
@@ -186,4 +264,12 @@
       <state_interface name="effort" />
     </joint>
+    <transmission name="trans_head_pan">
+      <plugin>transmission_interface/SimpleTransmission</plugin>
+      <actuator name="motor_head_pan" role="actuator1"/>
+      <joint name="joint_head_pan" role="joint1">
+          <mechanical_reduction>1.0</mechanical_reduction>
+          <offset>0.0</offset>
+      </joint>
+    </transmission>
     <joint name="joint_head_tilt">
       <command_interface name="position" />
@@ -194,4 +280,12 @@
       <state_interface name="effort" />
     </joint>
+    <transmission name="trans_head_tilt">
+      <plugin>transmission_interface/SimpleTransmission</plugin>
+      <actuator name="motor_head_tilt" role="actuator1"/>
+      <joint name="joint_head_tilt" role="joint1">
+          <mechanical_reduction>1.0</mechanical_reduction>
+          <offset>0.0</offset>
+      </joint>
+    </transmission>
   </ros2_control>
   <gazebo>

File: urdf/stretch_main.xacro (robot description, xacro)
@@ -210,5 +210,5 @@
         rpy="0 0 0" />
       <mass
-        value="0.18285" />
+        value="1.8285" />
       <inertia
         ixx="0.0709854511954588"
