Commit message: [Add]: Working version of stretch without manipulators

File: urdf/gazebo.urdf.xacro (robot description, xacro)
@@ -4,4 +4,8 @@
   <xacro:arg name="visualize_lidar" default="false" />
   <xacro:include filename="$(find stretch_gazebo)/urdf/stretch_main.xacro" />
+  <xacro:include filename="$(find stretch_gazebo)/urdf/stretch_gripper.xacro" />
+  <xacro:include filename="$(find stretch_gazebo)/urdf/stretch_aruco.xacro" />
+  <xacro:include filename="$(find stretch_gazebo)/urdf/stretch_respeaker.xacro" />
+  <xacro:include filename="$(find stretch_gazebo)/urdf/stretch_d435i.xacro" />
   <gazebo reference="base_link">
       <material>Gazebo/Gray</material>
@@ -110,21 +114,83 @@
       <minDepth>0.001</minDepth>
   </gazebo>
-  <ros2_control name="GazeboSimSystem" type="system">
+  <gazebo reference="link_gripper_finger_left">
+      <mu1 value="100.0"/>
+      <mu2 value="200.0"/>
+      <kp value="10000000.0" />
+      <kd value="100.0" />
+      <material>Gazebo/Gray</material>
+      <minDepth>0.001</minDepth>
+  </gazebo>
+  <gazebo reference="link_gripper_finger_right">
+      <mu1 value="100.0"/>
+      <mu2 value="200.0"/>
+      <kp value="10000000.0" />
+      <kd value="100.0" />
+      <material>Gazebo/Gray</material>
+      <minDepth>0.001</minDepth>
+  </gazebo>
+  <gazebo reference="link_grasp_center">
+      <mu1 value="100.0"/>
+      <mu2 value="200.0"/>
+      <kp value="10000000.0" />
+      <kd value="100.0" />
+      <material>Gazebo/Gray</material>
+      <minDepth>0.001</minDepth>
+  </gazebo>
+  <gazebo reference="link_gripper_fingertip_left">
+      <mu1 value="100.0"/>
+      <mu2 value="200.0"/>
+      <kp value="10000000.0" />
+      <kd value="100.0" />
+      <material>Gazebo/Black</material>
+      <minDepth>0.001</minDepth>
+  </gazebo>
+  <gazebo reference="link_gripper_fingertip_right">
+      <mu1 value="100.0"/>
+      <mu2 value="200.0"/>
+      <kp value="10000000.0" />
+      <kd value="100.0" />
+      <material>Gazebo/Black</material>
+      <minDepth>0.001</minDepth>
+  </gazebo>
+  <gazebo reference="link_gripper">
+      <mu1 value="100.0"/>
+      <mu2 value="200.0"/>
+      <kp value="10000000.0" />
+      <kd value="100.0" />
+      <material>Gazebo/Gray</material>
+      <minDepth>0.001</minDepth>
+  </gazebo>
+  <!-- Aruco -->
+  <gazebo reference="link_aruco_right_base">
+      <material>Gazebo/Black</material>
+  </gazebo>
+  <gazebo reference="link_aruco_left_base">
+      <material>Gazebo/Black</material>
+  </gazebo>
+  <gazebo reference="link_aruco_shoulder">
+      <material>Gazebo/Black</material>
+  </gazebo>
+  <gazebo reference="link_aruco_top_wrist">
+      <material>Gazebo/Black</material>
+  </gazebo>
+  <gazebo reference="link_aruco_inner_wrist">
+      <material>Gazebo/Black</material>
+  </gazebo>
+  <!-- Respeaker -->
+  <gazebo reference="respeaker_base">
+      <material>Gazebo/Green</material>
+  </gazebo>
+  <ros2_control name="GazeboSystem" type="system">
     <hardware>
       <plugin>gazebo_ros2_control/GazeboSystem</plugin>
     </hardware>
     <joint name="joint_right_wheel">
-      <command_interface name="velocity">
-        <param name="min">-0.5</param>
-        <param name="max">0.5</param>
-      </command_interface>
+      <command_interface name="velocity"/>
       <state_interface name="position" />
       <state_interface name="velocity" />
     </joint>
     <joint name="joint_left_wheel">
-        <command_interface name="velocity">
-          <param name="min">-0.5</param>
-          <param name="max">0.5</param>
-        </command_interface>
+        <command_interface name="velocity"/>
         <state_interface name="position" />
         <state_interface name="velocity" />
@@ -132,7 +198,7 @@
     <joint name="joint_lift">
       <command_interface name="position" />
-      <command_interface name="velocity" />
-      <command_interface name="effort" />
-      <state_interface name="position" />
+      <state_interface name="position">
+        <param name="initial_value">0.2</param>
+      </state_interface>
       <state_interface name="velocity" />
       <state_interface name="effort" />
@@ -140,6 +206,4 @@
     <joint name="joint_arm_l0">
       <command_interface name="position" />
-      <command_interface name="velocity" />
-      <command_interface name="effort" />
       <state_interface name="position" />
       <state_interface name="velocity" />
@@ -148,6 +212,4 @@
     <joint name="joint_arm_l1">
       <command_interface name="position" />
-      <command_interface name="velocity" />
-      <command_interface name="effort" />
       <state_interface name="position" />
       <state_interface name="velocity" />
@@ -156,6 +218,4 @@
     <joint name="joint_arm_l2">
       <command_interface name="position" />
-      <command_interface name="velocity" />
-      <command_interface name="effort" />
       <state_interface name="position" />
       <state_interface name="velocity" />
@@ -164,6 +224,4 @@
     <joint name="joint_arm_l3">
       <command_interface name="position" />
-      <command_interface name="velocity" />
-      <command_interface name="effort" />
       <state_interface name="position" />
       <state_interface name="velocity" />
@@ -172,7 +230,7 @@
     <joint name="joint_wrist_yaw">
       <command_interface name="position" />
-      <command_interface name="velocity" />
-      <command_interface name="effort" />
-      <state_interface name="position" />
+      <state_interface name="position">
+        <param name="initial_value">3.14</param>
+      </state_interface>
       <state_interface name="velocity" />
       <state_interface name="effort" />
@@ -180,6 +238,4 @@
     <joint name="joint_head_pan">
       <command_interface name="position" />
-      <command_interface name="velocity" />
-      <command_interface name="effort" />
       <state_interface name="position" />
       <state_interface name="velocity" />
@@ -188,6 +244,16 @@
     <joint name="joint_head_tilt">
       <command_interface name="position" />
-      <command_interface name="velocity" />
-      <command_interface name="effort" />
+      <state_interface name="position" />
+      <state_interface name="velocity" />
+      <state_interface name="effort" />
+    </joint>
+    <joint name="joint_gripper_finger_right">
+      <command_interface name="position" />
+      <state_interface name="position" />
+      <state_interface name="velocity" />
+      <state_interface name="effort" />
+    </joint>
+    <joint name="joint_gripper_finger_left">
+      <command_interface name="position" />
       <state_interface name="position" />
       <state_interface name="velocity" />

File: urdf/gazebo_base.urdf.xacro (robot description, xacro)
@@ -30,4 +30,36 @@
     <mu2>0.0</mu2>
   </gazebo>
+  <gazebo reference="link_mast">
+      <material>Gazebo/Gray</material>
+  </gazebo>
+  <gazebo reference="link_head">
+      <mu1 value="100.0"/>
+      <mu2 value="200.0"/>
+      <material>Gazebo/Gray</material>
+  </gazebo>
+  <gazebo reference="link_head_tilt">
+      <mu1 value="100.0"/>
+      <mu2 value="200.0"/>
+      <kp value="10000000.0" />
+      <kd value="100.0" />
+      <material>Gazebo/Gray</material>
+      <minDepth>0.001</minDepth>
+  </gazebo>
+  <gazebo reference="link_head_pan">
+      <mu1 value="100.0"/>
+      <mu2 value="200.0"/>
+      <kp value="10000000.0" />
+      <kd value="100.0" />
+      <material>Gazebo/Gray</material>
+      <minDepth>0.001</minDepth>
+  </gazebo>
+  <!-- <gazebo reference="link_lift">
+      <mu1 value="10000.0"/>
+      <mu2 value="10000.0"/>
+      <kp value="10000000.0" />
+      <kd value="100.0" />
+      <material>Gazebo/Black</material>
+      <minDepth>0.001</minDepth>
+  </gazebo> -->
   <ros2_control name="GazeboSystem" type="system">
     <hardware>
@@ -44,4 +76,22 @@
       <state_interface name="velocity"/>
     </joint>
+    <joint name="joint_head_pan">
+      <command_interface name="position" />
+      <state_interface name="position" />
+      <state_interface name="velocity" />
+      <state_interface name="effort" />
+    </joint>
+    <joint name="joint_head_tilt">
+      <command_interface name="position" />
+      <state_interface name="position" />
+      <state_interface name="velocity" />
+      <state_interface name="effort" />
+    </joint>
+    <!-- <joint name="joint_lift">
+      <command_interface name="position"/>
+      <state_interface name="position"/>
+      <state_interface name="velocity" />
+      <state_interface name="effort" />
+    </joint> -->
   </ros2_control>
   <gazebo>

File: urdf/stretch_base.xacro (robot description, xacro)
@@ -12,4 +12,7 @@
     <color rgba="1 1 1 1"/>
   </material>
+  <material name="black">
+    <color rgba="0.0 0.0 0.0 1.0"/>
+  </material>
   <xacro:macro name="default_inertial" params="mass pos">
     <inertial>
@@ -176,3 +179,264 @@
     <axis xyz="0 0 1" />
   </joint>
+  <link
+    name="link_mast">
+    <inertial>
+      <origin
+        xyz="2.0817E-17 0.7075 -2.7756E-17"
+        rpy="0 0 0" />
+      <mass
+        value="0.18285" />
+      <inertia
+        ixx="0.0709854511954588"
+        ixy="-0.00433428742758457"
+        ixz="-0.000186110788697573"
+        iyy="0.000437922053342648"
+        iyz="-0.00288788257713431"
+        izz="0.071104808501661" />
+    </inertial>
+    <visual>
+      <origin
+        xyz="0 0 0"
+        rpy="0 0 0" />
+      <geometry>
+        <mesh
+          filename="package://stretch_gazebo/meshes/link_mast.STL" />
+      </geometry>
+      <material name="white"/>
+    </visual>
+    <collision>
+      <origin
+        xyz="0 0 0"
+        rpy="0 0 0" />
+      <geometry>
+        <mesh
+          filename="package://stretch_gazebo/meshes/link_mast.STL" />
+      </geometry>
+    </collision>
+  </link>
+  <joint
+    name="joint_mast"
+    type="fixed">
+    <origin
+      xyz="-0.067 0.135 0.0284"
+      rpy="1.5708 0 4.8006E-17" />
+    <parent
+      link="base_link" />
+    <child
+      link="link_mast" />
+    <axis
+      xyz="0 0 0" />
+  </joint>
+  <link
+    name="link_head">
+    <inertial>
+      <origin
+        xyz="0.0406850995527703 0.0396956343318414 0.0226500246461012"
+        rpy="0 0 0" />
+      <mass
+        value="0.133027236718691" />
+      <inertia
+        ixx="0.001"
+        ixy="0"
+        ixz="0"
+        iyy="0.001"
+        iyz="0"
+        izz="0.001" />
+    </inertial>
+    <visual>
+      <origin
+        xyz="0 0 0"
+        rpy="0 0 0" />
+      <geometry>
+        <mesh
+          filename="package://stretch_gazebo/meshes/link_head.STL" />
+      </geometry>
+      <material
+        name="">
+        <color
+          rgba="0.792156862745098 0.819607843137255 0.933333333333333 1" />
+      </material>
+    </visual>
+    <collision>
+      <origin
+        xyz="0 0 0"
+        rpy="0 0 0" />
+      <geometry>
+        <mesh
+          filename="package://stretch_gazebo/meshes/link_head.STL" />
+      </geometry>
+    </collision>
+  </link>
+  <joint
+    name="joint_head"
+    type="fixed">
+    <origin
+      xyz="0 1.33 0"
+      rpy="1.5707963267949 -1.5707963267949 3.1416" />
+    <parent
+      link="link_mast" />
+    <child
+      link="link_head" />
+    <axis
+      xyz="0 0 0" />
+  </joint>
+  <link
+    name="link_head_pan">
+    <inertial>
+      <origin
+        xyz="-0.000326562615178591 0.00850012613776489 0.000130487222982367"
+        rpy="0 0 0" />
+      <mass
+        value="0.0273764496535409" />
+      <inertia
+        ixx="0.001"
+        ixy="0"
+        ixz="0"
+        iyy="0.001"
+        iyz="0"
+        izz="0.001" />
+    </inertial>
+    <visual>
+      <origin
+        xyz="0 0 0"
+        rpy="0 0 0" />
+      <geometry>
+        <mesh
+          filename="package://stretch_gazebo/meshes/link_head_pan.STL" />
+      </geometry>
+      <material
+        name="">
+        <color
+          rgba="0.792156862745098 0.819607843137255 0.933333333333333 1" />
+      </material>
+    </visual>
+    <collision>
+      <origin
+        xyz="0 0 0"
+        rpy="0 0 0" />
+      <geometry>
+        <mesh
+          filename="package://stretch_gazebo/meshes/link_head_pan.STL" />
+      </geometry>
+    </collision>
+  </link>
+  <joint
+    name="joint_head_pan"
+    type="revolute">
+    <origin
+      xyz="0.135 0.0731000000000001 -0.00319621125547975"
+      rpy="0 0 1.5707963267949" />
+    <parent
+      link="link_head" />
+    <child
+      link="link_head_pan" />
+    <axis
+      xyz="0 0 1" />
+    <limit effort="100" lower="-3.9" upper="1.5" velocity="1.0"/>
+  </joint>
+  <link
+    name="link_head_tilt">
+    <inertial>
+      <origin
+        xyz="0.00704566394917504 -0.0212256210929691 0.0302058990060359"
+        rpy="0 0 0" />
+      <mass
+        value="0.090217113313934" />
+      <inertia
+        ixx="0.001"
+        ixy="0"
+        ixz="0"
+        iyy="0.001"
+        iyz="0"
+        izz="0.001" />
+    </inertial>
+    <visual>
+      <origin
+        xyz="0 0 0"
+        rpy="0 0 0" />
+      <geometry>
+        <mesh
+          filename="package://stretch_gazebo/meshes/link_head_tilt.STL" />
+      </geometry>
+      <material
+        name="">
+        <color
+          rgba="0.792156862745098 0.819607843137255 0.933333333333333 1" />
+      </material>
+    </visual>
+    <collision>
+      <origin
+        xyz="0 0 0"
+        rpy="0 0 0" />
+      <geometry>
+        <mesh
+          filename="package://stretch_gazebo/meshes/link_head_tilt.STL" />
+      </geometry>
+    </collision>
+  </link>
+  <joint
+    name="joint_head_tilt"
+    type="revolute">
+    <origin
+      xyz="-0.00130000001785262 0.0277624999926072 -0.0533107920897029"
+      rpy="1.5707963267949 3.36459255518345E-15 -8.42914893687103E-17" />
+    <parent
+      link="link_head_pan" />
+    <child
+      link="link_head_tilt" />
+    <axis
+      xyz="0 0 1" />
+    <limit effort="100" lower="-1.53" upper="0.79" velocity="1.0"/>
+  </joint>
+  <!-- <link
+    name="link_lift">
+    <inertial>
+      <origin
+        xyz="-0.031727 0.038403 0.013361"
+        rpy="0 0 0" />
+      <mass
+        value="0.27218" />
+      <inertia
+        ixx="0.00052571"
+        ixy="0.00014899"
+        ixz="-1.9258E-05"
+        iyy="0.00030679"
+        iyz="-6.2451E-06"
+        izz="0.00037324" />
+    </inertial>
+    <visual>
+      <origin
+        xyz="0 0 0"
+        rpy="0 0 0" />
+      <geometry>
+        <mesh
+          filename="package://stretch_gazebo/meshes/link_lift.STL" />
+      </geometry>
+      <material name="black"/>
+    </visual>
+    <collision>
+      <origin
+        xyz="0 0 0"
+        rpy="0 0 0" />
+      <geometry>
+        <mesh
+          filename="package://stretch_gazebo/meshes/link_lift.STL" />
+      </geometry>
+    </collision>
+  </link>
+  <joint
+    name="joint_lift"
+    type="prismatic">
+    <origin
+      xyz="-0.037385 0.1666 0"
+      rpy="-1.5708 1.5708 0" />
+    <parent
+      link="link_mast" />
+    <child
+      link="link_lift" />
+    <axis
+      xyz="0 0 1" />
+    <limit effort="100" lower="0.001" upper="1.1" velocity="1.0"/>
+    <dynamics damping="0.1" friction="0.1"/>
+  </joint> -->
 </robot>

File: urdf/stretch_main.xacro (robot description, xacro)
@@ -2,6 +2,6 @@
 <robot xmlns:xacro="http://www.ros.org/wiki/xacro" name="stretch_main">
   <xacro:property name="M_PI" value="3.1415926535897931" />
-  <xacro:property name="joint_damping" value="0"/>
-  <xacro:property name="joint_friction" value="0"/>
+  <xacro:property name="joint_damping" value="0.0"/>
+  <xacro:property name="joint_friction" value="0.0"/>
   <xacro:property name="joint_spring_stiffness" value="0"/>
   <xacro:property name="joint_spring_reference" value="0"/>
