Commit message: [Add]: Working version of mobile base + head with sensors

File: urdf/stretch_main.xacro (robot description, xacro)
@@ -2,8 +2,32 @@
 <robot xmlns:xacro="http://www.ros.org/wiki/xacro" name="stretch_main">
   <xacro:property name="M_PI" value="3.1415926535897931" />
-  <xacro:property name="joint_damping" value="21.75"/>
-  <xacro:property name="joint_friction" value="10.48"/>
+  <xacro:property name="joint_damping" value="0"/>
+  <xacro:property name="joint_friction" value="0"/>
   <xacro:property name="joint_spring_stiffness" value="0"/>
   <xacro:property name="joint_spring_reference" value="0"/>
+  <material name="blue">
+    <color rgba="0 0 0.8 1"/>
+  </material>
+  <material name="white">
+    <color rgba="1 1 1 1"/>
+  </material>
+  <material name="black">
+    <color rgba="0.0 0.0 0.0 1.0"/>
+  </material>
+  <xacro:macro name="default_inertial" params="mass pos">
+    <inertial>
+      <origin
+        xyz="${pos}"
+        rpy="0 0 0" />
+      <mass value="${mass}" />
+      <inertia
+        ixx="0.01"
+        ixy="0"
+        ixz="0"
+        iyy="0.01"
+        iyz="0"
+        izz="0.01" />
+    </inertial>
+  </xacro:macro>
   <link
     name="base_link">
@@ -16,8 +40,8 @@
       <inertia
         ixx="0.0034667"
-        ixy="-5.0568E-06"
-        ixz="0.00042861"
+        ixy="0"
+        ixz="0"
         iyy="0.0052744"
-        iyz="-5.766E-05"
+        iyz="0"
         izz="0.0047945" />
     </inertial>
@@ -30,9 +54,5 @@
           filename="package://stretch_gazebo/meshes/base_link.STL" />
       </geometry>
-      <material
-        name="">
-        <color
-          rgba="0.79216 0.81961 0.93333 1" />
-      </material>
+       <material name="white"/>
     </visual>
     <collision>
@@ -48,18 +68,4 @@
   <link
     name="link_right_wheel">
-    <inertial>
-      <origin
-        xyz="1.1719E-11 2.0783E-11 0.037544"
-        rpy="0 0 0" />
-      <mass
-        value="0.0042721" />
-      <inertia
-        ixx="0.001"
-        ixy="0"
-        ixz="0"
-        iyy="0.001"
-        iyz="0"
-        izz="0.001" />
-    </inertial>
     <visual>
       <origin
@@ -70,9 +76,5 @@
           filename="package://stretch_gazebo/meshes/link_right_wheel.STL" />
       </geometry>
-      <material
-        name="">
-        <color
-          rgba="0.79216 0.81961 0.93333 1" />
-      </material>
+      <material name="blue"/>
     </visual>
     <collision>
@@ -85,4 +87,5 @@
       </geometry>
     </collision>
+    <xacro:default_inertial mass="0.0042721" pos="1.1719E-11 2.0783E-11 0.037544"/>
   </link>
   <joint
@@ -102,18 +105,4 @@
   <link
     name="link_left_wheel">
-    <inertial>
-      <origin
-        xyz="-2.0783E-11 -1.1719E-11 -0.037544"
-        rpy="0 0 0" />
-      <mass
-        value="0.0042721" />
-      <inertia
-        ixx="0.001"
-        ixy="0"
-        ixz="0"
-        iyy="0.001"
-        iyz="0"
-        izz="0.001" />
-    </inertial>
     <visual>
       <origin
@@ -124,9 +113,5 @@
           filename="package://stretch_gazebo/meshes/link_left_wheel.STL" />
       </geometry>
-      <material
-        name="">
-        <color
-          rgba="0.79216 0.81961 0.93333 1" />
-      </material>
+      <material name="blue"/>
     </visual>
     <collision>
@@ -139,4 +124,5 @@
       </geometry>
     </collision>
+    <xacro:default_inertial mass="0.0042721" pos="-2.0783E-11 -1.1719E-11 -0.037544"/>
   </link>
   <joint
@@ -185,15 +171,5 @@
       </material>
     </visual>
-    <inertial>
-      <mass value="0.01" />
-      <origin xyz="0 0 0" />
-      <inertia
-        ixx="0.001"
-        ixy="0"
-        ixz="0"
-        iyy="0.001"
-        iyz="0"
-        izz="0.001" />
-    </inertial>
+    <xacro:default_inertial mass="0.01" pos="0 0 0"/>
   </link>
   <joint name="caster_joint" type="fixed">
@@ -210,5 +186,5 @@
         rpy="0 0 0" />
       <mass
-        value="1.8285" />
+        value="0.18285" />
       <inertia
         ixx="0.0709854511954588"
@@ -227,9 +203,5 @@
           filename="package://stretch_gazebo/meshes/link_mast.STL" />
       </geometry>
-      <material
-        name="">
-        <color
-          rgba="0.79216 0.81961 0.93333 1" />
-      </material>
+      <material name="white"/>
     </visual>
     <collision>
@@ -257,118 +229,11 @@
   </joint>
   <link
-    name="link_lift">
-    <inertial>
-      <origin
-        xyz="-0.031727 0.038403 0.013361"
-        rpy="0 0 0" />
-      <mass
-        value="0.27218" />
-      <inertia
-        ixx="0.00052571"
-        ixy="0.00014899"
-        ixz="-1.9258E-05"
-        iyy="0.00030679"
-        iyz="-6.2451E-06"
-        izz="0.00037324" />
-    </inertial>
-    <visual>
-      <origin
-        xyz="0 0 0"
-        rpy="0 0 0" />
-      <geometry>
-        <mesh
-          filename="package://stretch_gazebo/meshes/link_lift.STL" />
-      </geometry>
-      <material
-        name="">
-        <color
-          rgba="0.79216 0.81961 0.93333 1" />
-      </material>
-    </visual>
-    <collision>
-      <origin
-        xyz="0 0 0"
-        rpy="0 0 0" />
-      <geometry>
-        <mesh
-          filename="package://stretch_gazebo/meshes/link_lift.STL" />
-      </geometry>
-    </collision>
-  </link>
-  <joint
-    name="joint_lift"
-    type="prismatic">
-    <origin
-      xyz="-0.037385 0.1666 0"
-      rpy="-1.5708 1.5708 0" />
-    <parent
-      link="link_mast" />
-    <child
-      link="link_lift" />
-    <axis
-      xyz="0 0 1" />
-  <limit effort="100" lower="0.0" upper="1.1" velocity="1.0"/>
-  </joint>
-  <link
-    name="link_arm_l4">
-    <inertial>
-      <origin
-        xyz="-1.0146E-06 -1.9719E-05 -0.094738"
-        rpy="0 0 0" />
-      <mass
-        value="0.068095" />
-      <inertia
-        ixx="0.0001256"
-        ixy="-5.6914E-12"
-        ixz="6.0647E-09"
-        iyy="0.0001256"
-        iyz="1.1787E-07"
-        izz="1.1091E-10" />
-    </inertial>
-    <visual>
-      <origin
-        xyz="0 0 0"
-        rpy="0 0 0" />
-      <geometry>
-        <mesh
-          filename="package://stretch_gazebo/meshes/link_arm_l4.STL" />
-      </geometry>
-      <material
-        name="">
-        <color
-          rgba="0.79216 0.81961 0.93333 1" />
-      </material>
-    </visual>
-    <collision>
-      <origin
-        xyz="0 0 0"
-        rpy="0 0 0" />
-      <geometry>
-        <mesh
-          filename="package://stretch_gazebo/meshes/link_arm_l4.STL" />
-      </geometry>
-    </collision>
-  </link>
-  <joint
-    name="joint_arm_l4"
-    type="fixed">
-    <origin
-      xyz="-0.2547 0 0"
-      rpy="1.5708 2.4721E-15 -1.5708" />
-    <parent
-      link="link_lift" />
-    <child
-      link="link_arm_l4" />
-    <axis
-      xyz="0 0 0" />
-  </joint>
-  <link
-    name="link_arm_l3">
-    <inertial>
-      <origin
-        xyz="-5.13853606326845E-07 -1.99844969271112E-05 -0.0971104963726614"
-        rpy="0 0 0" />
-      <mass
-        value="0.0628927381893134" />
+    name="link_head">
+    <inertial>
+      <origin
+        xyz="0.0406850995527703 0.0396956343318414 0.0226500246461012"
+        rpy="0 0 0" />
+      <mass
+        value="0.133027236718691" />
       <inertia
         ixx="0.001"
@@ -385,5 +250,5 @@
       <geometry>
         <mesh
-          filename="package://stretch_gazebo/meshes/link_arm_l3.STL" />
+          filename="package://stretch_gazebo/meshes/link_head.STL" />
       </geometry>
       <material
@@ -399,31 +264,29 @@
       <geometry>
         <mesh
-          filename="package://stretch_gazebo/meshes/link_arm_l3.STL" />
-      </geometry>
-    </collision>
-  </link>
-  <joint
-    name="joint_arm_l3"
-    type="prismatic">
-    <origin
-      xyz="0 0 0.013"
-      rpy="7.68831233799385E-30 2.36716479416092E-30 2.29652732251143E-17" />
-    <parent
-      link="link_arm_l4" />
-    <child
-      link="link_arm_l3" />
-    <axis
-      xyz="0 0 1" />
-    <!-- 0.13 = 0.52/4-->
-    <limit effort="100" lower="0.0" upper="0.13" velocity="1.0"/>
-  </joint>
-  <link
-    name="link_arm_l2">
-    <inertial>
-      <origin
-        xyz="-5.17421949435687E-07 -2.02045301450349E-05 -0.0968815475684904"
-        rpy="0 0 0" />
-      <mass
-        value="0.0571386353275368" />
+          filename="package://stretch_gazebo/meshes/link_head.STL" />
+      </geometry>
+    </collision>
+  </link>
+  <joint
+    name="joint_head"
+    type="fixed">
+    <origin
+      xyz="0 1.33 0"
+      rpy="1.5707963267949 -1.5707963267949 3.1416" />
+    <parent
+      link="link_mast" />
+    <child
+      link="link_head" />
+    <axis
+      xyz="0 0 0" />
+  </joint>
+  <link
+    name="link_head_pan">
+    <inertial>
+      <origin
+        xyz="-0.000326562615178591 0.00850012613776489 0.000130487222982367"
+        rpy="0 0 0" />
+      <mass
+        value="0.0273764496535409" />
       <inertia
         ixx="0.001"
@@ -440,5 +303,5 @@
       <geometry>
         <mesh
-          filename="package://stretch_gazebo/meshes/link_arm_l2.STL" />
+          filename="package://stretch_gazebo/meshes/link_head_pan.STL" />
       </geometry>
       <material
@@ -454,30 +317,30 @@
       <geometry>
         <mesh
-          filename="package://stretch_gazebo/meshes/link_arm_l2.STL" />
-      </geometry>
-    </collision>
-  </link>
-  <joint
-    name="joint_arm_l2"
-    type="prismatic">
-    <origin
-      xyz="0 0 0.013"
-      rpy="0 1.57655765344625E-30 -1.66533453693773E-16" />
-    <parent
-      link="link_arm_l3" />
-    <child
-      link="link_arm_l2" />
+          filename="package://stretch_gazebo/meshes/link_head_pan.STL" />
+      </geometry>
+    </collision>
+  </link>
+  <joint
+    name="joint_head_pan"
+    type="revolute">
+    <origin
+      xyz="0.135 0.0731000000000001 -0.00319621125547975"
+      rpy="0 0 1.5707963267949" />
+    <parent
+      link="link_head" />
+    <child
+      link="link_head_pan" />
     <axis
       xyz="0 0 1" />
-    <limit effort="100" lower="0.0" upper="0.13" velocity="1.0"/>
-  </joint>
-  <link
-    name="link_arm_l1">
-    <inertial>
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